Commit message: Update ros2_control.xacro
Controller for the cart still needs hardware interface

File: description/ros2_control.xacro (robot description, xacro)
@@ -1,8 +1,15 @@
 <?xml version="1.0"?>
 <robot xmlns:xacro="http://www.ros.org/wiki/xacro">
-  <ros2_control name="SmartSystem" type="system">
+  <ros2_control name="SmartCart" type="system">
         <hardware>
-            <plugin>smartcart_ros2_control/SmartSystem</plugin> <!--hardware interface-->
+            <plugin>smartcart_ros2_control/SmartSystem</plugin> <!--TO DO:hardware interface-->
         </hardware>
+        <param name="left_wheel_name">left_wheel_joint</param>
+        <param name="right_wheel_name">right_wheel_joint</param>
+        <param name="loop_rate"></param>                         <!--TO DO:find params-->
+        <param name="device"></param>
+        <param name="baud_rate"></param>
+        <param name="timeout"></param>
+        <param name="enc_counts_per_rev"></param>
         <joint name="left_wheel_joint">
             <command_interface name="velocity">
@@ -23,7 +30,34 @@
   </ros2_control>
   <smartcart>
-      <plugin name="smartcart_ros2_control" name="libsmartcart_ros2_control.so"> <!--tells smartcart to use ros2 control-->
+      <plugin name="gazebo_ros2_control" name="libgazebo_ros2_control.so"> <!--tells simulation to use ros2 control-->
           <parameters>$(find smart-cart)/config/smart_controllers.yaml</parameters>
       </plugin>
   </smartcart>
+  <!--Controller for simulation -->
+ <!-- <ros2_control name="GazeboSystem" type="system">
+        <hardware>
+            <plugin>gazebo_ros2_control/GazeboSystem</plugin> <!--hardware interface-->
+        </hardware>
+        <joint name="left_wheel_joint">
+            <command_interface name="velocity">
+                <param name="min">-10</param>
+                <param name="max">10</param>
+            </command_interface>
+            <state_interface name="velocity"/>
+            <state_interface name="position"/>
+        </joint>
+        <joint name="right_wheel_joint">
+            <command_interface name="velocity">
+                <param name="min">-10</param>
+                <param name="max">10</param>
+            </command_interface>
+            <state_interface name="velocity"/>
+            <state_interface name="position"/>
+        </joint>
+  </ros2_control> -->
+  <gazebo>
+      <plugin name="gazebo_ros2_control" name="libgazebo_ros2_control.so"> <!--tells simulation to use ros2 control-->
+          <parameters>$(find smart-cart)/config/smart_controllers.yaml</parameters>
+      </plugin>
+  </gazebo>
 </robot>
