Commit message: Updates for rviz simulation

File: description/robot.urdf.xacro (robot description, xacro)
@@ -1,14 +1,5 @@
 <?xml version="1.0"?>
-<robot xmlns:xacro="http://www.ros.org/wiki/xacro" name="robot">
-    <!-- toggle between gazebo sim and ros2 control -->
-    <xacro:arg name="use_ros2" default="true"/>
+<robot xmlns:xacro="http://www.ros.org/wiki/xacro"  name="robot">
     <xacro:include filename="robot_core.xacro" />
-    <xacro:if value="$(arg use_ros2)">
-        <xacro:include filename="ros2_control.xacro" />
-    </xacro:if>
-    <xacro:unless value="$(arg use_ros2)">
-        <xacro:include filename="gazebo_control.xacro" /> <!-- TODO: update rsp file 11:18-->
-    </xacro:unless>
-    <xacro:include filename="lidar.xacro" />
-    <xacro:include filename="camera.xacro" />
+    <xacro:include filename="gazebo_control.xacro" />
 </robot>

File: description/robot_core.xacro (robot description, xacro)
@@ -1,116 +1,157 @@
 <?xml version="1.0"?>
-<robot xmlns:xacro="http://www.ros.org/wiki/xacro">
-  <xacro:include filename="inertial_macros.xacro"/>
-  <material name="white">
-      <color rgba="1 1 1 1" />
-  </material>
-  <material name="orange">
-      <color rgba="1 0.3 0.1 1" />
-  </material>
-  <material name="blue">
-      <color rgba="0.2 0.2 1 1" />
-  </material>
-  <material name="black">
-      <color rgba="0 0 0 1" />
-  </material>
-  <!--base link center of drive wheels-->
-  <link name="base_link">
-  </link>
-  <!--chassis link-->
-  <joint name="chassis_joint" type="fixed">
-      <parent link="base_link"/>
-      <child link="chassis"/>
-      <!--just behind base link-->
-      <origin xyz="-0.1 0 0"/>
-  </joint>
-  <link name="chassis">
-      <visual>
-          <origin xyz="0.15 0 0.075"/>
-          <geometry>
-              <box size="0.3 0.3 0.15"/> <!--cart dimensions-->
-          </geometry>
-          <material name="white"/>
-      </visual>
-      <collision>
-          <origin xyz="0.15 0 0.075"/>
-          <geometry>
-              <box size="0.3 0.3 0.15"/> <!--cart dimensions-->
-          </geometry>
-      </collision>
-      <xacro:inertial_box mass="0.5" x="0.3" y="0.3" z="0.3">
-          <origin xyz="0.15 0 0.075" rpy="0 0 0"/>
-      </xacro:inertial_box>
-  </link>
-  <!--left wheel link-->
-  <joint name="left_wheel_joint" type="continuous">
-      <parent link="base_link"/>
-      <child link="left_wheel"/>
-      <origin xyz="0 0.175 0" rpy="-${pi/2} 0 0"/>
-      <axis xyz="0 0 1"/>
-  </joint>
-  <link name="left_wheel">
-      <visual>
-          <origin xyz="0.15 0 0.075"/>
-          <geometry>
-              <cylinder radius="0.05" length="0.04"/> <!--wheel dimensions-->
-          </geometry>
-          <material name="blue"/>
-      </visual>
-      <collisiom>
-          <origin xyz="0.15 0 0.075"/>
-          <geometry>
-              <cylinder radius="0.05" length="0.04"/> <!--wheel dimensions-->
-          </geometry>
-      </collision>
-      <xacro:inertial_cylinder mass="0.1" length="0.04" radius="0.05">
-          <origin xyz="0 0 0" rpy="0 0 0"/>
-      </xacro:inertial_cylinder>
-  </link>
-  <!--right wheel link-->
-  <joint name="right_wheel_joint" type="continuous">
-      <parent link="base_link"/>
-      <child link="right_wheel"/>
-      <origin xyz="0 -0.175 0" rpy="${pi/2} 0 0"/>
-      <axis xyz="0 0 -1"/>
-  </joint>
-  <link name="right_wheel">
-      <visual>
-          <origin xyz="0.15 0 0.075"/>
-          <geometry>
-              <cylinder radius="0.05" length="0.04"/> <!--wheel dimensions-->
-          </geometry>
-          <material name="blue"/>
-      </visual>
-      <collision>
-          <origin xyz="0.15 0 0.075"/>
-          <geometry>
-              <cylinder radius="0.05" length="0.04"/> <!--wheel dimensions-->
-          </geometry>
-      </collision>
-      <xacro:inertial_cylinder mass="0.1" length="0.04" radius="0.05">
-          <origin xyz="0 0 0" rpy="0 0 0"/>
-      </xacro:inertial_cylinder>
-  </link>
-  <!--caster wheel link-->
-  <joint name="caster_wheel_joint" type="fixed">
-      <parent link="chassis"/>
-      <child link="caster_wheel"/>
-      <origin xyz="0.24 0 0"/>
-  </joint>
-  <link name="caster_wheel">
-      <visual>
-          <geometry>
-              <sphere radius="0.05"/> <!--wheel dimensions-->
-          </geometry>
-          <material name="black"/>
-      </visual>
-      <collision>
-          <geometry>
-              <sphere radius="0.05"/> <!--wheel dimensions-->
-          </geometry>
-      </collision>
-      <xacro:inertial_sphere mass="0.1" radius="0.05">
-          <origin xyz="0 0 0" rpy="0 0 0"/>
-      </xacro:inertial_sphere>
-  </link>
+<robot xmlns:xacro="http://www.ros.org/wiki/xacro" >
+    <xacro:include filename="inertial_macros.xacro"/>
+    <material name="white">
+        <color rgba="1 1 1 1" />
+    </material>
+    <material name="orange">
+        <color rgba="1 0.3 0.1 1"/>
+    </material>
+    <material name="blue">
+        <color rgba="0.2 0.2 1 1"/>
+    </material>
+    <material name="black">
+        <color rgba="0 0 0 1"/>
+    </material>
+    <material name="gray">
+        <color rgba="0.5 0.5 0.5 0.5"/>
+    </material>
+    <!-- BASE LINK: center of cart -->
+    <link name="base_link">
+    </link>
+    <!-- CHASSIS LINK -->
+    <joint name="chassis_joint" type="fixed">
+        <parent link="base_link"/>
+        <child link="chassis"/>
+        <origin xyz="0 0 0"/>
+    </joint>
+    <link name="chassis">
+        <visual>
+            <origin xyz="0 0 0.4191"/>
+            <geometry>
+                <box size="1.143 0.635 0.8382"/>        <!-- Cart Dimensions-->
+            </geometry>
+            <material name="gray"/>
+        </visual>
+        <collision>
+            <origin xyz="0 0 0.4191"/>
+            <geometry>
+                <box size="1.143 0.635 0.8382"/>        <!-- Cart Dimensions-->
+            </geometry>
+        </collision>
+        <xacro:inertial_box mass="19.5" x="1.143" y="0.635" z="0.8382">
+            <origin xyz="0.5715 0 0.04191" rpy="0 0 0"/>
+        </xacro:inertial_box>
+    </link>
+    <gazebo reference="chassis">
+        <material>Gazebo/Gray</material>
+    </gazebo>
+    <!-- LEFT DRIVER WHEEL LINK -->
+    <joint name="left_wheel_joint" type="continuous">
+        <parent link="base_link"/>
+        <child link="left_wheel"/>
+        <origin xyz="0.257175 0.254 0" rpy="-${pi/2} 0 0" />
+        <axis xyz="0 0 1"/>
+    </joint>
+    <link name="left_wheel">
+        <visual>
+            <geometry>
+                <cylinder radius="0.127" length="0.04"/>
+            </geometry>
+            <material name="blue"/>
+        </visual>
+        <collision>
+            <geometry>
+                <cylinder radius="0.127" length="0.04"/>
+            </geometry>
+        </collision>
+        <xacro:inertial_cylinder mass="0.1" length="0.04" radius="0.127">
+            <origin xyz="0 0 0" rpy="0 0 0"/>
+        </xacro:inertial_cylinder>
+    </link>
+    <gazebo reference="left_wheel">
+        <material>Gazebo/Blue</material>
+    </gazebo>
+    <!-- RIGHT DRIVER WHEEL LINK -->
+    <joint name="right_wheel_joint" type="continuous">
+        <parent link="base_link"/>
+        <child link="right_wheel"/>
+        <origin xyz="0.257175 -0.254 0" rpy="${pi/2} 0 0" />
+        <axis xyz="0 0 -1"/>
+    </joint>
+    <link name="right_wheel">
+        <visual>
+            <geometry>
+                <cylinder radius="0.127" length="0.04"/>
+            </geometry>
+            <material name="blue"/>
+        </visual>
+        <collision>
+            <geometry>
+                <cylinder radius="0.127" length="0.04"/>
+            </geometry>
+        </collision>
+        <xacro:inertial_cylinder mass="0.1" length="0.04" radius="0.127">
+            <origin xyz="0 0 0" rpy="0 0 0"/>
+        </xacro:inertial_cylinder>
+    </link>
+    <gazebo reference="right_wheel">
+        <material>Gazebo/Blue</material>
+    </gazebo>
+    <!-- LEFT FIXED WHEEL LINK -->
+    <joint name="left_fixed_wheel_joint" type="continuous">
+        <parent link="base_link"/>
+        <child link="left_fixed_wheel"/>
+        <origin xyz="-0.257175 0.254 0" rpy="-${pi/2} 0 0" />
+        <axis xyz="0 0 1"/>
+    </joint>
+    <link name="left_fixed_wheel">
+        <visual>
+            <geometry>
+                <cylinder radius="0.127" length="0.04"/>
+            </geometry>
+            <material name="blue"/>
+        </visual>
+        <collision>
+            <geometry>
+                <cylinder radius="0.127" length="0.04"/>
+            </geometry>
+        </collision>
+        <xacro:inertial_cylinder mass="0.1" length="0.04" radius="0.127">
+            <origin xyz="0 0 0" rpy="0 0 0"/>
+        </xacro:inertial_cylinder>
+    </link>
+    <gazebo reference="left_fixed_wheel">
+        <material>Gazebo/Blue</material>
+        <mu1 value="0.001"/>                  <!--friction coefficients-->
+        <mu2 value="0.001"/>
+    </gazebo>
+    <!-- RIGHT FIXED WHEEL LINK -->
+    <joint name="right_fixed_wheel_joint" type="continuous">
+        <parent link="base_link"/>
+        <child link="right_fixed_wheel"/>
+        <origin xyz="-0.257175  -0.254 0" rpy="${pi/2} 0 0" />
+        <axis xyz="0 0 -1"/>
+    </joint>
+    <link name="right_fixed_wheel">
+        <visual>
+            <geometry>
+                <cylinder radius="0.127" length="0.04"/>
+            </geometry>
+            <material name="blue"/>
+        </visual>
+        <collision>
+            <geometry>
+                <cylinder radius="0.127" length="0.04"/>
+            </geometry>
+        </collision>
+        <xacro:inertial_cylinder mass="0.1" length="0.04" radius="0.127">
+            <origin xyz="0 0 0" rpy="0 0 0"/>
+        </xacro:inertial_cylinder>
+    </link>
+    <gazebo reference="right_fixed_wheel">
+        <material>Gazebo/Blue</material>
+        <mu1 value="0.001"/>                    <!--friction coefficients-->
+        <mu2 value="0.001"/>
+    </gazebo>
 </robot>
